File: Testing/4-bit R2R DAC/Schematics/4-bit R2R DAC.kicad_sch (KiCad schematic)
At the start: 0 parts

Commit message: Schematics Update
Parts:
- added D1, D2, D3, D4: LED, LED_THT:LED_D3.0mm_Clear, symbol Device:LED
- added J1: SpeakON_NL2, Connector_Audio:Jack_speakON_Neutrik_NL2MDXX-V_Vertical, symbol Connector_Audio:SpeakON_NL2
- added Q1: 2N2219, Package_TO_SOT_THT:TO-39-3, symbol Transistor_BJT:2N2219
- added R1, R10, R11, R12, R13, R2, R3, R4, R5, R6, R7, R8, R9: R, Resistor_THT:R_Axial_DIN0204_L3.6mm_D1.6mm_P5.08mm_Horizontal, symbol Device:R
- added RV1: R_Potentiometer_Trim_US, Potentiometer_THT:Potentiometer_Bourns_3296W_Vertical, symbol Device:R_Potentiometer_Trim_US
- added U1: ESP32-DEVKITC-32E, ESP32:MODULE_ESP32-DEVKITC-32E, symbol ESP32-DEVKITC-32E:ESP32-DEVKITC-32E
- added U2: DM-OLED096-636, DM-OLED096-636:MODULE_DM-OLED096-636, symbol DM-OLED096-636:DM-OLED096-636
Connections:
- new net: R3.1, R7.1, U1.J3_10 (IO5)
- new net: R10.2, R11.1, R7.2
- new net: R4.1, R8.1, U1.J3_11 (IO17)
- new net: D4.2 (A), R4.2
- new net: D1.1 (K), D2.1 (K), D3.1 (K), D4.1 (K), Q1.1 (E), R12.2, RV1.1, U1.J3_1 (GND_J3_1), U2.1 (GND)
- new net: RV1.2, U1.J2_6 (IO35)
- new net: RV1.3, U1.J2_1 (3V3), U2.2 (VCC_IN)
- new net: Q1.2 (B), R13.1
- new net: J1.1-, Q1.3 (C)
- new net: R13.2, R5.1, R9.1, U1.J2_5 (IO34)
- new net: R10.1, R6.2, R9.2
- new net: J1.1+, U1.J2_19 (EXT_5V)
- new net: R11.2, R12.1, R8.2
- new net: D1.2 (A), R1.2
- new net: U1.J3_3 (IO22), U2.3 (SCL)
- new net: U1.J3_6 (IO21), U2.4 (SDA)
- new net: R1.1, R5.2, U1.J3_8 (IO19)
- new net: R2.1, R6.1, U1.J3_9 (IO18)
- new net: D3.2 (A), R3.2
- new net: D2.2 (A), R2.2
- no-connect marks 0 -> 27
